File: kicad/chihuahua.kicad_sch (KiCad schematic)
At the start: 41 parts, among them J1 CARTRIDGE, J2 VIAport, J3 IOx, J4 nanoLink, J5 STEP, J6 POWER, Q1 BC548, Q2 BC548, SW1 RESET, SW2 NMI, U1 65C02, U2 65C22, U3 62256, U4 74HC132, U5 74HC32, X1 1 MHz

Commit message: v1.3
Parts:
- removed C2: 0, Capacitor_THT:CP_Radial_D4.0mm_P1.50mm, symbol chihuahua-rescue:CP-Device
- removed D2: 1N4148, Diode_THT:D_DO-35_SOD27_P2.54mm_Vertical_AnodeUp, symbol Device:D
- added Q3: BC548, Package_TO_SOT_THT:TO-92_Inline, symbol Transistor_BJT:BC548
- R4: value 3K3 -> 680
Connections:
- net +5V: now also U4.1, U4.2, Q3.1 (C); no longer SW2.2
- net CB2: now also Q3.2 (B); no longer BZ1.1 (-), U5.1, U5.2, U5.3, U5.4, U5.5, U5.6
- net GND: now also SW2.1; no longer R4.2
- net PB7: now also U5.1, U5.2, U5.4, U5.5; no longer U5.8
- net U_RST: now also R4.2; no longer C1.2, U4.4, U4.5
- net ~{NMI}: now also SW2.2; no longer U4.3
- net D_PB7 renamed BPB7
- net BPB7: now also U5.3, U5.6, U5.8
- removed net U_NMI: R4.1, SW2.1, U4.1, U4.2
- new net BCB2: BZ1.1 (-), Q3.3 (E)
- new net RST: C1.2, R4.1, U4.4, U4.5
- no-connect marks 13 -> 14
Other:
- note added: "~{IOC}"
- moved on the sheet: H1, H2, H3, R3, R4, SW1, SW2, U4A, U5A, U5B
